File: 0-24V_PWM_Buck/0-24VBuck/0-24VBuck.sch (KiCad schematic (older format))
At the start: 57 parts, among them J1 Output, Q1 TIP122, Q10 PN2907, Q11 PN2907, Q12 PN2222, Q13 PN2222, Q14 PN2222, Q15 PN2222, Q16 PN2907, Q17 PMOS_50V_100A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

Commit message: Update Circuit Image
Update Circuit Image
Parts:
- R10, R5: value 4.7K -> 10K
- R13: value 4K -> 1k
- R6, R9: value 10k -> 100k
Connections:
- net at Q15.3 (E), Q16.3 (E), R16.2: no longer D9.2 (A)
- net at Q17.2 (G), R15.2, R16.1: now also D9.2 (A)
Other:
- moved on the sheet: D9
Changed lines of the file:
@@
 P 5250 6550
 F 0 "R5" V 5330 6550 50  0000 C CNN
-F 1 "4.7K" V 5250 6550 50  0000 C CNN
+F 1 "10K" V 5250 6550 50  0000 C CNN
 F 2 "" V 5180 6550 50  0000 C CNN
 F 3 "" H 5250 6550 50  0000 C CNN
@@
 P 5700 5500
 F 0 "R6" V 5780 5500 50  0000 C CNN
-F 1 "10k" V 5700 5500 50  0000 C CNN
+F 1 "100k" V 5700 5500 50  0000 C CNN
 F 2 "" V 5630 5500 50  0000 C CNN
 F 3 "" H 5700 5500 50  0000 C CNN
@@
 P 9100 6550
 F 0 "R10" V 9180 6550 50  0000 C CNN
-F 1 "4.7K" V 9100 6550 50  0000 C CNN
+F 1 "10K" V 9100 6550 50  0000 C CNN
 F 2 "" V 9030 6550 50  0000 C CNN
 F 3 "" H 9100 6550 50  0000 C CNN
@@
 P 8650 5500
 F 0 "R9" V 8730 5500 50  0000 C CNN
-F 1 "10k" V 8650 5500 50  0000 C CNN
+F 1 "100k" V 8650 5500 50  0000 C CNN
 F 2 "" V 8580 5500 50  0000 C CNN
 F 3 "" H 8650 5500 50  0000 C CNN
@@
 P 10650 5550
 F 0 "R13" V 10730 5550 50  0000 C CNN
-F 1 "4K" V 10650 5550 50  0000 C CNN
+F 1 "1k" V 10650 5550 50  0000 C CNN
 F 2 "" V 10580 5550 50  0000 C CNN
 F 3 "" H 10650 5550 50  0000 C CNN
@@
 Wire Wire Line
 	8650 5750 8650 6000
-$Comp
-L Device:D_Zener D9
-U 1 1 5FCF7403
-P 12500 4350
-F 0 "D9" H 12500 4450 50  0000 C CNN
-F 1 "12v" H 12500 4250 50  0000 C CNN
-F 2 "" H 12500 4350 50  0000 C CNN
-F 3 "" H 12500 4350 50  0000 C CNN
-	1    12500 4350
-	0    1    1    0
-$EndComp
 Wire Wire Line
 	11950 4450 11950 4650
-Wire Wire Line
-	11600 3950 12500 3950
 Connection ~ 11600 3950
-Wire Wire Line
-	11950 4650 12500 4650
 Connection ~ 11950 4650
 Wire Wire Line
 	11950 4650 11950 4800
-Wire Wire Line
-	12500 4500 12500 4650
-Connection ~ 12500 4650
-Wire Wire Line
-	12500 4650 13100 4650
-Wire Wire Line
-	12500 4200 12500 3950
-Connection ~ 12500 3950
-Wire Wire Line
-	12500 3950 12750 3950
 Wire Wire Line
 	11950 6700 13500 6700
@@
 	850  5300 850  6700
 Connection ~ 1400 6700
+$Comp
+L Device:D_Zener D9
+U 1 1 5FCF7403
+P 12500 4200
+F 0 "D9" H 12500 4300 50  0000 C CNN
+F 1 "12v" H 12500 4100 50  0000 C CNN
+F 2 "" H 12500 4200 50  0000 C CNN
+F 3 "" H 12500 4200 50  0000 C CNN
+	1    12500 4200
+	0    1    1    0
+$EndComp
+Wire Wire Line
+	11600 3950 12500 3950
+Wire Wire Line
+	11950 4650 13100 4650
+Wire Wire Line
+	12500 4350 12750 4350
+Connection ~ 12750 4350
+Wire Wire Line
+	12500 4050 12500 3950
+Connection ~ 12500 3950
+Wire Wire Line
+	12500 3950 12750 3950
 $EndSCHEMATC
