File: SuperProject/SawOscillator.kicad_sch (KiCad schematic)
At the start: 8 parts

Commit message: Update Controller
Update Controller
Parts:
- removed C?: 1n, symbol Device:C
Connections:
- net C: now reaches D?.2 (A), Q?.2 (C), Q?.3 (E)
- net VCC: now reaches R?.1
- net GND: now reaches Q?.3 (E), R?.2
Changed lines of the file:
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@@
 (kicad_sch (version 20211123) (generator eeschema)
   (paper "A4")
+  (junction (at 139.7 77.47) (diameter 0) (color 0 0 0 0)
+  )
   (junction (at 151.13 90.17) (diameter 0) (color 0 0 0 0)
   )
   (junction (at 162.56 77.47) (diameter 0) (color 0 0 0 0)
   )
-  (junction (at 151.13 111.76) (diameter 0) (color 0 0 0 0)
+  (junction (at 162.56 111.76) (diameter 0) (color 0 0 0 0)
   )
   (junction (at 156.21 99.06) (diameter 0) (color 0 0 0 0)
-  )
-  (junction (at 128.27 77.47) (diameter 0) (color 0 0 0 0)
-  )
-  (junction (at 139.7 77.47) (diameter 0) (color 0 0 0 0)
   )
   (junction (at 162.56 90.17) (diameter 0) (color 0 0 0 0)
@@
     (stroke (width 0) (type default) (color 0 0 0 0))
   )
+  (wire (pts (xy 162.56 111.76) (xy 165.1 111.76))
+    (stroke (width 0) (type default) (color 0 0 0 0))
+  )
   (wire (pts (xy 162.56 97.79) (xy 162.56 99.06))
     (stroke (width 0) (type default) (color 0 0 0 0))
   )
-  (wire (pts (xy 128.27 111.76) (xy 128.27 95.25))
+  (wire (pts (xy 162.56 67.31) (xy 162.56 68.58))
     (stroke (width 0) (type default) (color 0 0 0 0))
   )
-  (wire (pts (xy 151.13 111.76) (xy 128.27 111.76))
+  (wire (pts (xy 165.1 67.31) (xy 162.56 67.31))
     (stroke (width 0) (type default) (color 0 0 0 0))
   )
@@
     (stroke (width 0) (type default) (color 0 0 0 0))
   )
-  (wire (pts (xy 128.27 77.47) (xy 128.27 87.63))
-    (stroke (width 0) (type default) (color 0 0 0 0))
-  )
   (wire (pts (xy 139.7 104.14) (xy 139.7 106.68))
     (stroke (width 0) (type default) (color 0 0 0 0))
@@
     (stroke (width 0) (type default) (color 0 0 0 0))
   )
+  (wire (pts (xy 139.7 74.93) (xy 139.7 77.47))
+    (stroke (width 0) (type default) (color 0 0 0 0))
+  )
+  (wire (pts (xy 135.89 77.47) (xy 139.7 77.47))
+    (stroke (width 0) (type default) (color 0 0 0 0))
+  )
   (wire (pts (xy 152.4 85.09) (xy 156.21 85.09))
     (stroke (width 0) (type default) (color 0 0 0 0))
   )
   (wire (pts (xy 162.56 111.76) (xy 162.56 107.95))
-    (stroke (width 0) (type default) (color 0 0 0 0))
-  )
-  (wire (pts (xy 128.27 77.47) (xy 125.73 77.47))
     (stroke (width 0) (type default) (color 0 0 0 0))
   )
@@
     (stroke (width 0) (type default) (color 0 0 0 0))
   )
-  (wire (pts (xy 162.56 67.31) (xy 162.56 68.58))
-    (stroke (width 0) (type default) (color 0 0 0 0))
-  )
-  (wire (pts (xy 139.7 77.47) (xy 128.27 77.47))
-    (stroke (width 0) (type default) (color 0 0 0 0))
-  )
   (wire (pts (xy 139.7 77.47) (xy 139.7 90.17))
     (stroke (width 0) (type default) (color 0 0 0 0))
@@
   (wire (pts (xy 162.56 76.2) (xy 162.56 77.47))
     (stroke (width 0) (type default) (color 0 0 0 0))
+  )
+  (hierarchical_label "C" (shape bidirectional) (at 139.7 74.93 90)
+    (effects (font (size 1.27 1.27)) (justify left))
+  )
+  (hierarchical_label "VOut" (shape output) (at 135.89 77.47 180)
+    (effects (font (size 1.27 1.27)) (justify right))
+  )
+  (hierarchical_label "GND" (shape output) (at 165.1 111.76 0)
+    (effects (font (size 1.27 1.27)) (justify left))
+  )
+  (hierarchical_label "VCC" (shape input) (at 165.1 67.31 0)
+    (effects (font (size 1.27 1.27)) (justify left))
   )
   (symbol (lib_id "Device:Q_PNP_BCE") (at 152.4 80.01 90) (unit 1)
@@
     (pin "1")
     (pin "2")
-  )
-  (symbol (lib_id "Device:C") (at 128.27 91.44 0) (unit 1)
-    (in_bom yes) (on_board yes)
-    (property "Reference" "C?" (id 0) (at 128.905 88.9 0)
-      (effects (font (size 1.27 1.27)) (justify left))
-    )
-    (property "Value" "1n" (id 1) (at 128.905 93.98 0)
-      (effects (font (size 1.27 1.27)) (justify left))
-    )
-    (property "Footprint" "" (id 2) (at 129.2352 95.25 0))
-    (property "Datasheet" "" (id 3) (at 128.27 91.44 0))
-    (pin "1")
-    (pin "2")
