File: SuperProject/OPAMP_C1.kicad_sch (KiCad schematic)
At the start: 16 parts

Commit message: Update Controller
Update Controller
Parts:
- removed C?: 1n, symbol Device:C
- removed D? (x2): 4148, symbol Device:D
- removed Q?: MMBT2222, symbol Device:Q_NPN_BCE
- removed Q?: MMBT2907, symbol Device:Q_PNP_BCE
- removed R? (x2): 4.7, symbol Device:R
- R? (x2): value 20k -> 10k
Connections:
- net VOut: now also Q?.2 (C), R?.2
Other:
- moved on the sheet: R?

Commit message: MPPT Complete
Parts:
- removed Q? (x3): MMBT2907, symbol Device:Q_PNP_BCE
- removed Q? (x2): MMBT2222, symbol Device:Q_NPN_BCE
- removed R? (x2): 10k, symbol Device:R
- removed R? (x2): 1k, symbol Device:R
- added Q? (x3): MMBT2907, symbol Device:Q_PNP_BCE
- added Q? (x2): MMBT2222, symbol Device:Q_NPN_BCE
- added R? (x2): 1k, symbol Device:R
- added R? (x2): 10k, symbol Device:R
Connections:
- net GND: now also R?.1, R?.1
- net V+: now also R?.1
- net V-: now also R?.1
- net VCC: now also Q?.3 (E), Q?.3 (E), Q?.3 (E)
- net VOut: now also Q?.2 (C), R?.2
- new net: Q?.1 (B), R?.2 (x2)
- new net: Q?.1 (B), Q?.1 (B), Q?.2 (C), Q?.2 (C)
- new net: Q?.3 (E), Q?.3 (E), R?.2
- new net: Q?.1 (B), Q?.2 (C), Q?.2 (C)
Changed lines of the file:
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@@
     (effects (font (size 1.27 1.27)) (justify right))
   )
-  (symbol (lib_id "Device:Q_PNP_BCE") (at 129.54 86.36 180) (unit 1)
+  (symbol (lib_id "Device:R") (at 170.18 111.76 180) (unit 1)
     (in_bom yes) (on_board yes)
-    (property "Reference" "Q?" (id 0) (at 121.92 85.09 90)
+    (property "Reference" "R?" (id 0) (at 168.91 113.03 0)
       (effects (font (size 1.27 1.27)) (justify left))
     )
-    (property "Value" "MMBT2907" (id 1) (at 124.46 81.28 90)
+    (property "Value" "1k" (id 1) (at 168.91 110.49 0)
       (effects (font (size 1.27 1.27)) (justify left))
     )
-    (property "Footprint" "" (id 2) (at 124.46 88.9 0)
+    (property "Footprint" "" (id 2) (at 171.958 111.76 90)
       (effects (font (size 1.27 1.27)) hide)
     )
-    (property "Datasheet" "~" (id 3) (at 129.54 86.36 0)
+    (property "Datasheet" "~" (id 3) (at 170.18 111.76 0)
       (effects (font (size 1.27 1.27)) hide)
     )
     (pin "1")
     (pin "2")
-    (pin "3")
   )
-  (symbol (lib_id "Device:Q_NPN_BCE") (at 165.1 106.68 0) (mirror y) (unit 1)
+  (symbol (lib_id "Device:Q_PNP_BCE") (at 160.02 80.01 0) (mirror x) (unit 1)
     (in_bom yes) (on_board yes)
-    (property "Reference" "Q?" (id 0) (at 157.48 107.95 90)
+    (property "Reference" "Q?" (id 0) (at 167.64 78.74 90)
       (effects (font (size 1.27 1.27)) (justify left))
     )
-    (property "Value" "MMBT2222" (id 1) (at 160.02 111.76 90)
+    (property "Value" "MMBT2907" (id 1) (at 165.1 74.93 90)
       (effects (font (size 1.27 1.27)) (justify left))
     )
-    (property "Footprint" "" (id 2) (at 160.02 104.14 0)
+    (property "Footprint" "" (id 2) (at 165.1 82.55 0)
       (effects (font (size 1.27 1.27)) hide)
     )
-    (property "Datasheet" "~" (id 3) (at 165.1 106.68 0)
-      (effects (font (size 1.27 1.27)) hide)
-    )
-    (pin "1")
-    (pin "2")
-    (pin "3")
-  )
-  (symbol (lib_id "Device:Q_PNP_BCE") (at 147.32 80.01 180) (unit 1)
-    (in_bom yes) (on_board yes)
-    (property "Reference" "Q?" (id 0) (at 139.7 78.74 90)
-      (effects (font (size 1.27 1.27)) (justify left))
-    )
-    (property "Value" "MMBT2907" (id 1) (at 142.24 74.93 90)
-      (effects (font (size 1.27 1.27)) (justify left))
-    )
-    (property "Footprint" "" (id 2) (at 142.24 82.55 0)
-      (effects (font (size 1.27 1.27)) hide)
-    )
-    (property "Datasheet" "~" (id 3) (at 147.32 80.01 0)
+    (property "Datasheet" "~" (id 3) (at 160.02 80.01 0)
       (effects (font (size 1.27 1.27)) hide)
     )
@@
     (pin "2")
   )
-  (symbol (lib_id "Device:R") (at 127 111.76 180) (unit 1)
+  (symbol (lib_id "Device:Q_NPN_BCE") (at 142.24 106.68 0) (unit 1)
     (in_bom yes) (on_board yes)
-    (property "Reference" "R?" (id 0) (at 125.73 113.03 0)
+    (property "Reference" "Q?" (id 0) (at 149.86 107.95 90)
       (effects (font (size 1.27 1.27)) (justify left))
     )
-    (property "Value" "10k" (id 1) (at 125.73 110.49 0)
+    (property "Value" "MMBT2222" (id 1) (at 147.32 111.76 90)
       (effects (font (size 1.27 1.27)) (justify left))
     )
-    (property "Footprint" "" (id 2) (at 128.778 111.76 90)
+    (property "Footprint" "" (id 2) (at 147.32 104.14 0)
       (effects (font (size 1.27 1.27)) hide)
     )
-    (property "Datasheet" "~" (id 3) (at 127 111.76 0)
+    (property "Datasheet" "~" (id 3) (at 142.24 106.68 0)
       (effects (font (size 1.27 1.27)) hide)
     )
     (pin "1")
     (pin "2")
+    (pin "3")
   )
   (symbol (lib_id "Device:R") (at 137.16 111.76 180) (unit 1)
@@
     (pin "2")
   )
-  (symbol (lib_id "Device:Q_PNP_BCE") (at 160.02 80.01 0) (mirror x) (unit 1)
+  (symbol (lib_id "Device:Q_PNP_BCE") (at 147.32 80.01 180) (unit 1)
     (in_bom yes) (on_board yes)
-    (property "Reference" "Q?" (id 0) (at 167.64 78.74 90)
+    (property "Reference" "Q?" (id 0) (at 139.7 78.74 90)
       (effects (font (size 1.27 1.27)) (justify left))
     )
-    (property "Value" "MMBT2907" (id 1) (at 165.1 74.93 90)
+    (property "Value" "MMBT2907" (id 1) (at 142.24 74.93 90)
       (effects (font (size 1.27 1.27)) (justify left))
     )
-    (property "Footprint" "" (id 2) (at 165.1 82.55 0)
+    (property "Footprint" "" (id 2) (at 142.24 82.55 0)
       (effects (font (size 1.27 1.27)) hide)
     )
-    (property "Datasheet" "~" (id 3) (at 160.02 80.01 0)
+    (property "Datasheet" "~" (id 3) (at 147.32 80.01 0)
       (effects (font (size 1.27 1.27)) hide)
     )
@@
     (pin "3")
   )
-  (symbol (lib_id "Device:Q_NPN_BCE") (at 142.24 106.68 0) (unit 1)
+  (symbol (lib_id "Device:Q_PNP_BCE") (at 129.54 86.36 180) (unit 1)
     (in_bom yes) (on_board yes)
-    (property "Reference" "Q?" (id 0) (at 149.86 107.95 90)
+    (property "Reference" "Q?" (id 0) (at 121.92 85.09 90)
       (effects (font (size 1.27 1.27)) (justify left))
     )
-    (property "Value" "MMBT2222" (id 1) (at 147.32 111.76 90)
+    (property "Value" "MMBT2907" (id 1) (at 124.46 81.28 90)
       (effects (font (size 1.27 1.27)) (justify left))
     )
-    (property "Footprint" "" (id 2) (at 147.32 104.14 0)
+    (property "Footprint" "" (id 2) (at 124.46 88.9 0)
       (effects (font (size 1.27 1.27)) hide)
     )
-    (property "Datasheet" "~" (id 3) (at 142.24 106.68 0)
+    (property "Datasheet" "~" (id 3) (at 129.54 86.36 0)
       (effects (font (size 1.27 1.27)) hide)
     )
@@
     (pin "3")
   )
-  (symbol (lib_id "Device:R") (at 170.18 111.76 180) (unit 1)
+  (symbol (lib_id "Device:R") (at 127 111.76 180) (unit 1)
     (in_bom yes) (on_board yes)
-    (property "Reference" "R?" (id 0) (at 168.91 113.03 0)
+    (property "Reference" "R?" (id 0) (at 125.73 113.03 0)
       (effects (font (size 1.27 1.27)) (justify left))
     )
-    (property "Value" "1k" (id 1) (at 168.91 110.49 0)
+    (property "Value" "10k" (id 1) (at 125.73 110.49 0)
       (effects (font (size 1.27 1.27)) (justify left))
     )
-    (property "Footprint" "" (id 2) (at 171.958 111.76 90)
+    (property "Footprint" "" (id 2) (at 128.778 111.76 90)
       (effects (font (size 1.27 1.27)) hide)
     )
-    (property "Datasheet" "~" (id 3) (at 170.18 111.76 0)
+    (property "Datasheet" "~" (id 3) (at 127 111.76 0)
       (effects (font (size 1.27 1.27)) hide)
     )
@@
     (pin "2")
   )
+  (symbol (lib_id "Device:Q_NPN_BCE") (at 165.1 106.68 0) (mirror y) (unit 1)
+    (in_bom yes) (on_board yes)
+    (property "Reference" "Q?" (id 0) (at 157.48 107.95 90)
+      (effects (font (size 1.27 1.27)) (justify left))
+    )
+    (property "Value" "MMBT2222" (id 1) (at 160.02 111.76 90)
+      (effects (font (size 1.27 1.27)) (justify left))
+    )
+    (property "Footprint" "" (id 2) (at 160.02 104.14 0)
+      (effects (font (size 1.27 1.27)) hide)
+    )
+    (property "Datasheet" "~" (id 3) (at 165.1 106.68 0)
+      (effects (font (size 1.27 1.27)) hide)
+    )
+    (pin "1")
+    (pin "2")
+    (pin "3")
+  )
   (sheet_instances
