File: SuperProject/OPAMP_N1.kicad_sch (KiCad schematic)
At the start: 16 parts

Commit message: MPPT Complete
Parts:
- removed C?: 1n, symbol Device:C
- removed D? (x2): 4148, symbol Device:D
- removed Q? (x4): MMBT2907, symbol Device:Q_PNP_BCE
- removed Q? (x3): MMBT2222, symbol Device:Q_NPN_BCE
- removed R? (x2): 20k, symbol Device:R
- removed R? (x2): 4.7, symbol Device:R
- removed R? (x2): 1k, symbol Device:R
- added C?: 1n, symbol Device:C
- added D? (x2): 4148, symbol Device:D
- added Q? (x3): MMBT2222, symbol Device:Q_NPN_BCE
- added Q? (x4): MMBT2907, symbol Device:Q_PNP_BCE
- added R? (x2): 1k, symbol Device:R
- added R? (x2): 4.7, symbol Device:R
- added R? (x2): 20k, symbol Device:R
Connections:
- net GND: now also Q?.2 (C), R?.1, R?.1
- net V+: now also R?.1
- net V-: now also R?.1
- net VCC: now also Q?.2 (C), Q?.3 (E), Q?.3 (E), Q?.3 (E)
- net VOut: now also R?.1, R?.2
- new net: Q?.1 (B), R?.2 (x2)
- new net: C?.2, Q?.1 (B), Q?.2 (C), Q?.2 (C)
- new net: Q?.3 (E), Q?.3 (E), R?.2
- new net: Q?.3 (E), R?.1
- new net: Q?.1 (B), Q?.1 (B), Q?.2 (C), Q?.2 (C)
- new net: C?.1, D?.2 (A), Q?.1 (B), Q?.2 (C)
- new net: D?.1 (K), Q?.1 (B), R?.2
- new net: Q?.3 (E), R?.2
- new net: D?.1 (K), D?.2 (A)
