File: SuperProject/SEPIC_10A_HS.kicad_sch (KiCad schematic)
At the start: 21 parts

Commit message: MPPT Complete
Parts:
- removed D?: MBRB10100, symbol Device:D_Schottky
- removed D?: 30SQ045, symbol Device:D_Schottky
Connections:
- net VOut: now also R?.4
Changed lines of the file:
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@@
   (junction (at 156.21 100.33) (diameter 0) (color 0 0 0 0)
   )
-  (junction (at 120.65 69.85) (diameter 0) (color 0 0 0 0)
-  )
   (junction (at 139.7 135.89) (diameter 0) (color 0 0 0 0)
   )
@@
     (stroke (width 0) (type default) (color 0 0 0 0))
   )
-  (wire (pts (xy 120.65 68.58) (xy 120.65 69.85))
-    (stroke (width 0) (type default) (color 0 0 0 0))
-  )
   (wire (pts (xy 156.21 83.82) (xy 156.21 85.09))
     (stroke (width 0) (type default) (color 0 0 0 0))
@@
     (stroke (width 0) (type default) (color 0 0 0 0))
   )
-  (wire (pts (xy 120.65 69.85) (xy 120.65 71.12))
-    (stroke (width 0) (type default) (color 0 0 0 0))
-  )
   (wire (pts (xy 139.7 101.6) (xy 139.7 111.76))
     (stroke (width 0) (type default) (color 0 0 0 0))
   )
-  (wire (pts (xy 116.84 69.85) (xy 120.65 69.85))
-    (stroke (width 0) (type default) (color 0 0 0 0))
-  )
   (wire (pts (xy 144.78 100.33) (xy 144.78 116.84))
     (stroke (width 0) (type default) (color 0 0 0 0))
@@
     (stroke (width 0) (type default) (color 0 0 0 0))
   )
-  (wire (pts (xy 120.65 101.6) (xy 128.27 101.6))
+  (wire (pts (xy 123.19 101.6) (xy 128.27 101.6))
     (stroke (width 0) (type default) (color 0 0 0 0))
   )
@@
     (stroke (width 0) (type default) (color 0 0 0 0))
   )
-  (wire (pts (xy 120.65 78.74) (xy 120.65 101.6))
-    (stroke (width 0) (type default) (color 0 0 0 0))
-  )
   (wire (pts (xy 163.83 134.62) (xy 163.83 135.89))
     (stroke (width 0) (type default) (color 0 0 0 0))
@@
     (stroke (width 0) (type default) (color 0 0 0 0))
   )
-  (wire (pts (xy 116.84 60.96) (xy 120.65 60.96))
+  (wire (pts (xy 123.19 67.31) (xy 123.19 101.6))
     (stroke (width 0) (type default) (color 0 0 0 0))
   )
@@
     (effects (font (size 1.27 1.27)) (justify left))
   )
-  (hierarchical_label "VBatt" (shape bidirectional) (at 116.84 69.85 180)
-    (effects (font (size 1.27 1.27)) (justify right))
-  )
   (hierarchical_label "VCS+" (shape output) (at 116.84 109.22 180)
     (effects (font (size 1.27 1.27)) (justify right))
@@
     (effects (font (size 1.27 1.27)) (justify left))
   )
-  (hierarchical_label "VOut" (shape output) (at 116.84 60.96 180)
-    (effects (font (size 1.27 1.27)) (justify right))
+  (hierarchical_label "VOut" (shape output) (at 123.19 67.31 90)
+    (effects (font (size 1.27 1.27)) (justify left))
   )
   (hierarchical_label "VFB" (shape output) (at 116.84 123.19 180)
@@
     (pin "3")
   )
-  (symbol (lib_id "Device:D_Schottky") (at 120.65 74.93 270) (unit 1)
-    (in_bom yes) (on_board yes)
-    (property "Reference" "D?" (id 0) (at 127 74.6125 0))
-    (property "Value" "MBRB10100" (id 1) (at 124.46 74.6125 0))
-    (property "Footprint" "" (id 2) (at 120.65 74.93 0)
-      (effects (font (size 1.27 1.27)) hide)
-    )
-    (property "Datasheet" "~" (id 3) (at 120.65 74.93 0)
-      (effects (font (size 1.27 1.27)) hide)
-    )
-    (pin "1")
-    (pin "2")
-  )
   (symbol (lib_id "Device:Q_NMOS_DGS") (at 161.29 116.84 0) (unit 1)
     (in_bom yes) (on_board yes)
@@
       (effects (font (size 1.27 1.27)) hide)
     )
-    (pin "1")
-    (pin "2")
-  )
-  (symbol (lib_id "Device:D_Schottky") (at 120.65 64.77 270) (unit 1)
-    (in_bom yes) (on_board yes)
-    (property "Reference" "D?" (id 0) (at 125.73 63.5 90)
-      (effects (font (size 1.27 1.27)) (justify left))
-    )
-    (property "Value" "30SQ045" (id 1) (at 123.19 65.7224 90)
-      (effects (font (size 1.27 1.27)) (justify left))
-    )
-    (property "Footprint" "" (id 2) (at 120.65 64.77 0)
-      (effects (font (size 1.27 1.27)) hide)
-    )
-    (property "Datasheet" "~" (id 3) (at 120.65 64.77 0)
-      (effects (font (size 1.27 1.27)) hide)
-    )
