File: SuperProject/MPPT.kicad_sch (KiCad schematic)
At the start: 25 parts

Commit message: Update Controller
Update Controller
Parts:
- added C?: 220p, symbol Device:C
- added C?: 1000u, symbol Device:C
- added D?: G, symbol Device:LED
- added D?: 5.1v, symbol Device:D_Zener
- added D?: 6.8v, symbol Device:D_Zener
- added Q? (x4): MMBT2222, symbol Device:Q_NPN_BCE
- added R? (x3): 1k, symbol Device:R
- added R? (x6): 10k, symbol Device:R
- added R?: 1, symbol Device:R
- added RV? (x2): 10k, symbol Device:R_Potentiometer
Connections:
- net GND: now also C?.1, C?.1, D?.2 (A), D?.2 (A), R?.2, R?.2, R?.2, R?.2, RV?.1, RV?.1
- net SEPIC/VFB: now also D?.1 (K)
- net SEPIC/VTH: now also Q?.3 (E), R?.1, RV?.3, RV?.3
- net UCS1/VCC: now also Q?.2 (C), Q?.2 (C), Q?.2 (C), Q?.2 (C), R?.1, R?.1
- net UVI/V-: now reaches RV?.2
- net UCS1/V_Out renamed UCS1/VOut
- net UCS2/V_Out renamed UCS2/VOut
- new net: D?.2 (A), R?.1
- new net: Q?.3 (E), R?.1, R?.2
- new net: D?.1 (K), Q?.1 (B), R?.2 (x2)
- new net: Q?.1 (B), R?.2 (x2)
- new net: Q?.3 (E), R?.1
- new net: C?.2, R?.1
- new net SawOscillator/C: C?.2
- new net SawOscillator/VCC: Q?.3 (E), R?.1
- new net SawOscillator/VOut: R?.1, R?.1
- new net UVI/VOut: R?.2
Other:
- added sheet UVI (OPAMP_C1.kicad_sch)
- sheet SawOscillator ports: added C, GND, VCC, VOut; removed none
- sheet UCS1 ports: added VOut; removed V_Out
- sheet UCS2 ports: added VOut; removed V_Out

Commit message: MPPT Complete
Parts:
- removed C?: 1000u, symbol Device:C
- added C?: 470u, symbol Device:C_Polarized
- added C?: 470p, symbol Device:C
- added C? (x3): 15p, symbol Device:C
- added C? (x3): 1000u, symbol Device:C_Polarized
- added C? (x3): 22n, symbol Device:C
- added C?: 10u, symbol Device:C_Polarized
- added D?: Y, symbol Device:LED
- added D? (x4): 4148, symbol Device:D
- added D?: SS34, symbol Device:D_Schottky
- added D?: MBRB10100, symbol Device:D_Schottky
- added D?: B, symbol Device:LED
- added D?: 30SQ045, symbol Device:D_Schottky
- added D? (x2): R, symbol Device:LED
- added D?: G, symbol Device:LED
- added D?: 5.1v, symbol Device:D_Zener
- added D?: 9.1v, symbol Device:D_Zener
- added Q? (x10): MMBT2222, symbol Device:Q_NPN_BCE
- added Q?: AOD403, symbol Device:Q_PMOS_DGS
- added Q?: AO3404, symbol Device:Q_NMOS_DGS
- added Q?: MMBT2907, symbol Device:Q_PNP_BCE
- added R? (x12): 1k, symbol Device:R
- added R? (x8): 4.7k, symbol Device:R
- added R? (x3): 330k, symbol Device:R
- added R? (x2): 100, symbol Device:R
- added R? (x7): 10k, symbol Device:R
- added R?: 680, symbol Device:R
- added R? (x2): 6.2k, symbol Device:R
- added R?: 560, symbol Device:R
- added R?: 510, symbol Device:R
- added R?: 0.025, symbol Device:R_Shunt
- added R?: 620, symbol Device:R
- added RV? (x3): 10k, symbol Device:R_Potentiometer
- added TH?: 24V 2A, symbol Device:Thermistor_PTC
- added TH?: 10K, symbol Device:Thermistor_NTC
Connections:
- net GND: now also C?.2, C?.2, C?.2, C?.2, C?.2, C?.2, D?.2 (A), Q?.2 (C), Q?.3 (E), Q?.3 (E), Q?.3 (E), Q?.3 (E), Q?.3 (E), Q?.3 (E), Q?.3 (E), Q?.3 (E), Q?.3 (S), R?.2, R?.2, R?.2, R?.2, R?.2, R?.2, R?.2, RV?.1, RV?.1, RV?.3, TH?.2
- net SEPIC/VFB: now also R?.1
- net SEPIC/VOut: now also D?.2 (A); no longer D?.1 (K)
- net SEPIC/VSW: now also Q?.3 (E), Q?.3 (E)
- net SEPIC/VTH: now also R?.2; no longer Q?.3 (E), R?.1, RV?.3, RV?.3
- net SawOscillator/VCC: now also Q?.3 (E), R?.1, RV?.3, RV?.3, R?.1
- net VBatt: now also D?.1 (K), D?.2 (A)
- net at Q?.3 (E), R?.1, R?.2: now also R?.1
- net at C?.1, Q?.3 (E), R?.1: now also R?.1
- net at Q?.3 (E), R?.1: now also R?.1
- net UError2/V+: now reaches RV?.2
- net UTEMP1/V+: now reaches RV?.2
- net UDRIMOS/V-: now reaches Q?.3 (E), R?.1
- net at R?.1: now also C?.1
- net UTEMP2/V-: now reaches RV?.2
- net UCS1/VCC renamed NOR/VCC
- net NOR/VCC: now also Q?.2 (C), R?.1, R?.2
- net ULEDINDC/V- renamed UError3/V+
- new net: D?.1 (K), Q?.2 (C) (x5)
- new net: D?.2 (A), R?.2 (x4)
- new net: Q?.1 (B), R?.2 (x3)
- new net: R?.1, R?.2 (x4)
- new net: C?.1, D?.1 (K), Q?.2 (C), Q?.2 (C), R?.2
- new net: C?.2, R?.2 (x3)
- new net: Q?.2 (G), R?.1, R?.2 (x2)
- new net: Q?.2 (C), R?.2
- new net: C?.1, Q?.1 (B), R?.2
- new net: Q?.3 (E), R?.1, R?.1, RV?.3, RV?.3
- new net: Q?.1 (B), R?.1, R?.2 (x4)
- new net: D?.2 (A), R?.1, R?.1
- new net: C?.1, D?.1 (K), D?.1 (K), R?.1
- new net: D?.1 (K), Q?.1 (B), R?.2
- new net: D?.2 (A), R?.1
- new net NOR/B: R?.1
- new net NOR/VOut: Q?.1 (B), Q?.1 (B)
- new net RS1/Q: R?.1, R?.1
- new net RS2/Q: R?.1
- new net UBUFF/V+: D?.2 (A), D?.2 (A), D?.2 (A), D?.2 (A), R?.2
- new net UBUFF/V-: RV?.1
- new net UDRIMOS/V+: RV?.2
- new net UError1/V-: C?.2, R?.1, R?.2
- new net UError1/VOut: C?.1, C?.1, D?.1 (K)
- new net UError2/V-: C?.2, R?.1, R?.2
- new net UError2/VOut: C?.1, C?.1, D?.1 (K)
- new net UError3/V-: C?.2, R?.1, R?.2
- new net UError3/VOut: C?.1, C?.1, D?.1 (K)
- new net UTEMP3/V+: RV?.2
- new net UTEMP3/V-: R?.2, TH?.1
- new net UTEMP4/V-: RV?.2
- new net VCS+: R?.2
- new net VCS-: R?.3
- new net VFAN+: C?.1, D?.1 (K), Q?.1 (D), Q?.2 (C), R?.1, R?.1, R?.1, R?.1, R?.1, R?.1, R?.1, R?.1, R?.1, TH?.2
- new net VFAN-: D?.2 (A), Q?.1 (D)
- new net VINSW: D?.1 (K)
- new net VOutCtrl: C?.1, TH?.1
- new net VOutPWR: Q?.3 (S), R?.1, R?.4
- no-connect marks 0 -> 3
Other:
- sheet UVI renamed ULEDINDC
- added sheet NOR (RTL_NOR.kicad_sch)
- added sheet NOT (RTL_NOT.kicad_sch)
- added sheet RS1 (RTL_RS.kicad_sch)
- added sheet RS2 (RTL_RS.kicad_sch)
- added sheet UBUFF (OPAMP_S1.kicad_sch)
- added sheet UDRIMOS (OPAMP_C1.kicad_sch)
- added sheet UError1 (OPAMP_S1.kicad_sch)
- added sheet UError2 (OPAMP_S1.kicad_sch)
- added sheet UError3 (OPAMP_S1.kicad_sch)
- added sheet UTEMP1 (OPAMP_C1.kicad_sch)
- added sheet UTEMP2 (OPAMP_C1.kicad_sch)
- added sheet UTEMP3 (OPAMP_C1.kicad_sch)
- added sheet UTEMP4 (OPAMP_C1.kicad_sch)
- added sheet UVLOASTABLE (UVLOASTABLE.kicad_sch)
- sheet SEPIC: file MPPT_SEPIC.kicad_sch -> SEPIC_10A_HS.kicad_sch
- sheet SEPIC ports: added none; removed VBatt
- moved on the sheet: C?, D?, F?, Q?, R?, RV?

Commit message: Update Zener
Parts:
- removed R? (x3): 4.7k, symbol Device:R
- added D?: 10v, symbol Device:D_Zener
- added D?: 11v, symbol Device:D_Zener
- added D?: 12v, symbol Device:D_Zener
- D?: value Y -> G
- D?: value B -> R
- D?: value G -> Y
- D?: value R -> B
- R? (x4): value 4.7k -> 1k
- R?: value 680 -> 10k
- R?: value 560 -> 10k
- R?: value 510 -> 10k
- R?: value 4.7k -> 1
- R?: value 620 -> 10k
Connections:
- net at R?.2: now also D?.1 (K) (x3)
- net at Q?.1 (B), R?.1: now also D?.2 (A) (x3)
Changed lines of the file:
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@@
       (effects (font (size 1.27 1.27)) (justify left))
     )
-    (property "Value" "Y" (id 1) (at 149.86 38.4174 90)
+    (property "Value" "G" (id 1) (at 149.86 38.4174 90)
       (effects (font (size 1.27 1.27)) (justify left))
     )
@@
       (effects (font (size 1.27 1.27)) (justify left))
     )
-    (property "Value" "4.7k" (id 1) (at 123.19 27.9399 0)
+    (property "Value" "1k" (id 1) (at 123.19 27.9399 0)
       (effects (font (size 1.27 1.27)) (justify left))
     )
@@
       (effects (font (size 1.27 1.27)) (justify left))
     )
-    (property "Value" "B" (id 1) (at 185.42 38.4174 90)
+    (property "Value" "R" (id 1) (at 185.42 38.4174 90)
       (effects (font (size 1.27 1.27)) (justify left))
     )
@@
       (effects (font (size 1.27 1.27)) (justify left))
     )
-    (property "Value" "680" (id 1) (at 123.19 55.8799 0)
+    (property "Value" "10k" (id 1) (at 123.19 55.8799 0)
       (effects (font (size 1.27 1.27)) (justify left))
     )
@@
     )
     (property "Datasheet" "~" (id 3) (at 120.65 54.61 0)
+      (effects (font (size 1.27 1.27)) hide)
+    )
+    (pin "1")
+    (pin "2")
+  )
+  (symbol (lib_id "Device:D_Zener") (at 156.21 36.83 270) (unit 1)
+    (in_bom yes) (on_board yes)
+    (property "Reference" "D?" (id 0) (at 158.75 35.5599 90)
+      (effects (font (size 1.27 1.27)) (justify left))
+    )
+    (property "Value" "10v" (id 1) (at 158.75 38.1 90)
+      (effects (font (size 1.27 1.27)) (justify left))
+    )
+    (property "Footprint" "" (id 2) (at 156.21 36.83 0)
+      (effects (font (size 1.27 1.27)) hide)
+    )
+    (property "Datasheet" "~" (id 3) (at 156.21 36.83 0)
       (effects (font (size 1.27 1.27)) hide)
     )
@@
       (effects (font (size 1.27 1.27)) (justify left))
     )
-    (property "Value" "4.7k" (id 1) (at 158.75 27.9399 0)
+    (property "Value" "1k" (id 1) (at 158.75 27.9399 0)
       (effects (font (size 1.27 1.27)) (justify left))
     )
@@
       (effects (font (size 1.27 1.27)) (justify left))
     )
-    (property "Value" "560" (id 1) (at 158.75 55.8799 0)
+    (property "Value" "10k" (id 1) (at 158.75 55.8799 0)
       (effects (font (size 1.27 1.27)) (justify left))
     )
@@
       (effects (font (size 1.27 1.27)) (justify left))
     )
-    (property "Value" "510" (id 1) (at 176.53 55.8799 0)
+    (property "Value" "10k" (id 1) (at 176.53 55.8799 0)
       (effects (font (size 1.27 1.27)) (justify left))
     )
@@
       (effects (font (size 1.27 1.27)) (justify left))
     )
-    (property "Value" "G" (id 1) (at 167.64 38.4174 90)
+    (property "Value" "Y" (id 1) (at 167.64 38.4174 90)
       (effects (font (size 1.27 1.27)) (justify left))
     )
@@
     (pin "2")
   )
-  (symbol (lib_id "Device:R") (at 120.65 36.83 0) (unit 1)
-    (in_bom yes) (on_board yes) (fields_autoplaced)
-    (property "Reference" "R?" (id 0) (at 123.19 35.5599 0)
-      (effects (font (size 1.27 1.27)) (justify left))
-    )
-    (property "Value" "4.7k" (id 1) (at 123.19 38.0999 0)
-      (effects (font (size 1.27 1.27)) (justify left))
-    )
-    (property "Footprint" "" (id 2) (at 118.872 36.83 90)
-      (effects (font (size 1.27 1.27)) hide)
-    )
-    (property "Datasheet" "~" (id 3) (at 120.65 36.83 0)
-      (effects (font (size 1.27 1.27)) hide)
-    )
-    (pin "1")
-    (pin "2")
-  )
   (symbol (lib_id "Device:C_Polarized") (at 191.77 43.18 0) (unit 1)
     (in_bom yes) (on_board yes)
@@
       (effects (font (size 1.27 1.27)) (justify left))
     )
-    (property "Value" "4.7k" (id 1) (at 176.53 27.9399 0)
+    (property "Value" "1k" (id 1) (at 176.53 27.9399 0)
       (effects (font (size 1.27 1.27)) (justify left))
     )
@@
       (effects (font (size 1.27 1.27)) (justify left))
     )
-    (property "Value" "R" (id 1) (at 132.08 38.4174 90)
+    (property "Value" "B" (id 1) (at 132.08 38.4174 90)
       (effects (font (size 1.27 1.27)) (justify left))
     )
@@
     (pin "2")
   )
-  (symbol (lib_id "Device:R") (at 156.21 36.83 0) (unit 1)
-    (in_bom yes) (on_board yes) (fields_autoplaced)
-    (property "Reference" "R?" (id 0) (at 158.75 35.5599 0)
-      (effects (font (size 1.27 1.27)) (justify left))
-    )
-    (property "Value" "4.7k" (id 1) (at 158.75 38.0999 0)
-      (effects (font (size 1.27 1.27)) (justify left))
-    )
-    (property "Footprint" "" (id 2) (at 154.432 36.83 90)
-      (effects (font (size 1.27 1.27)) hide)
-    )
-    (property "Datasheet" "~" (id 3) (at 156.21 36.83 0)
-      (effects (font (size 1.27 1.27)) hide)
-    )
-    (pin "1")
-    (pin "2")
-  )
   (symbol (lib_id "Device:Q_PNP_BCE") (at 273.05 120.65 0) (mirror x) (unit 1)
     (in_bom yes) (on_board yes)
@@
       (effects (font (size 1.27 1.27)) (justify left))
     )
-    (property "Value" "4.7k" (id 1) (at 176.53 38.0999 0)
+    (property "Value" "1" (id 1) (at 176.53 38.0999 0)
       (effects (font (size 1.27 1.27)) (justify left))
     )
@@
       (effects (font (size 1.27 1.27)) (justify left))
     )
-    (property "Value" "620" (id 1) (at 140.97 55.8799 0)
+    (property "Value" "10k" (id 1) (at 140.97 55.8799 0)
       (effects (font (size 1.27 1.27)) (justify left))
     )
@@
     (pin "2")
   )
+  (symbol (lib_id "Device:D_Zener") (at 138.43 36.83 270) (unit 1)
+    (in_bom yes) (on_board yes)
+    (property "Reference" "D?" (id 0) (at 140.97 35.5599 90)
+      (effects (font (size 1.27 1.27)) (justify left))
+    )
+    (property "Value" "11v" (id 1) (at 140.97 38.1 90)
+      (effects (font (size 1.27 1.27)) (justify left))
+    )
+    (property "Footprint" "" (id 2) (at 138.43 36.83 0)
+      (effects (font (size 1.27 1.27)) hide)
+    )
+    (property "Datasheet" "~" (id 3) (at 138.43 36.83 0)
+      (effects (font (size 1.27 1.27)) hide)
+    )
+    (pin "1")
+    (pin "2")
+  )
   (symbol (lib_id "Device:R") (at 119.38 81.28 0) (unit 1)
     (in_bom yes) (on_board yes)
@@
       (effects (font (size 1.27 1.27)) (justify left))
     )
-    (property "Value" "4.7k" (id 1) (at 140.97 27.9399 0)
+    (property "Value" "1k" (id 1) (at 140.97 27.9399 0)
       (effects (font (size 1.27 1.27)) (justify left))
     )
@@
     (pin "3")
   )
-  (symbol (lib_id "Device:R") (at 138.43 36.83 0) (unit 1)
-    (in_bom yes) (on_board yes) (fields_autoplaced)
-    (property "Reference" "R?" (id 0) (at 140.97 35.5599 0)
-      (effects (font (size 1.27 1.27)) (justify left))
-    )
-    (property "Value" "4.7k" (id 1) (at 140.97 38.0999 0)
-      (effects (font (size 1.27 1.27)) (justify left))
-    )
-    (property "Footprint" "" (id 2) (at 136.652 36.83 90)
-      (effects (font (size 1.27 1.27)) hide)
-    )
-    (property "Datasheet" "~" (id 3) (at 138.43 36.83 0)
-      (effects (font (size 1.27 1.27)) hide)
-    )
-    (pin "1")
-    (pin "2")
-  )
   (symbol (lib_id "Device:D_Schottky") (at 270.51 39.37 0) (unit 1)
     (in_bom yes) (on_board yes) (fields_autoplaced)
@@
       (effects (font (size 1.27 1.27)) hide)
     )
+    (pin "1")
+    (pin "2")
+  )
+  (symbol (lib_id "Device:D_Zener") (at 120.65 36.83 270) (unit 1)
+    (in_bom yes) (on_board yes)
+    (property "Reference" "D?" (id 0) (at 123.19 35.5599 90)
+      (effects (font (size 1.27 1.27)) (justify left))
+    )
+    (property "Value" "12v" (id 1) (at 123.19 38.1 90)
+      (effects (font (size 1.27 1.27)) (justify left))
+    )
+    (property "Footprint" "" (id 2) (at 120.65 36.83 0)
+      (effects (font (size 1.27 1.27)) hide)
+    )
+    (property "Datasheet" "~" (id 3) (at 120.65 36.83 0)
+      (effects (font (size 1.27 1.27)) hide)
+    )
